File: HW/hd6303-mb-ram-rom-x1-ext-dec.sch (EAGLE design)
At the start: 37 parts, among them IC1 74HC138N, IC2 AM29F010N

Commit message: fixes
Parts:
- added C11, C12, C13, C14, C15, C16: 10uF, resistor:C-EUC0805
- added C17: 100n, rcl:C-EUC0603
- added U2: (no value), MicroUSB:USB""
Connections:
- net +5V: now also C11.1, C12.1, C13.1, C14.1, C15.1, C16.1, C17.1, U2.VBUS
- net GND: now also C11.2, C12.2, C13.2, C14.2, C15.2, C16.2, C17.2, U2.GND
