File: HW/hd6303-mb-ram-rom-x1-ext-dec.brd (EAGLE design)
At the start: 100 x 80 mm, 37 parts, among them IC1 74HC138N, IC2 AM29F010N

Commit message: traced pcb
Routing:
- net +5V: track 0.00 -> 261.2 mm
- net IRQ1: track 0.00 -> 173.2 mm, vias 0 -> 2
- net WR: track 0.00 -> 155.9 mm, vias 0 -> 1
- net A6: track 0.00 -> 136.4 mm, vias 0 -> 2
- net A12: track 0.00 -> 133.9 mm
- net IRQ2: track 0.00 -> 130.9 mm, vias 0 -> 2
- net A5: track 0.00 -> 129.9 mm, vias 0 -> 2
- net A7: track 0.00 -> 129.7 mm, vias 0 -> 2
- net RES: track 0.00 -> 124.1 mm
- net NMI: track 0.00 -> 122.6 mm, vias 0 -> 4
- net MEM_A15: track 0.00 -> 120.7 mm, vias 0 -> 3
- net RD: track 0.00 -> 113.9 mm, vias 0 -> 2
- net PAGE_A15: track 0.00 -> 108.1 mm, vias 0 -> 1
- net PAGE_FN1: track 0.00 -> 106.1 mm, vias 0 -> 2
- net MEM_A16: track 0.00 -> 104.2 mm, vias 0 -> 2
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
Commit message: fixes
Parts:
- added C11, C12, C13, C14, C15, C16: 10uF, resistor:C0805
- added C17: 100n, rcl:C0603
- added U2: (no value), MicroUSB:USB-MICRO-SMD
- moved U$12 27.4 mm to (31.8, 74.9), turned to 180 degrees
- moved C2 19.4 mm to (3.81, 59.7), turned to 0 degrees
- moved R10 13.0 mm to (17.8, 73.7), turned to 270 degrees
- moved C3 12.5 mm to (16.5, 57.1), turned to 180 degrees
- moved C1 12.5 mm to (3.81, 64.8), turned to 0 degrees
- moved Q1 10.9 mm to (7.62, 62.2), turned to 90 degrees
- moved R6 7.62 mm to (16.5, 59.7)
- moved LED1 5.68 mm to (21.6, 74.9), turned to 0 degrees
- moved R4 5.08 mm to (16.5, 52.1)
- moved R5 5.08 mm to (16.5, 54.6)
- moved U$1 4.02 mm to (21.6, 36.8)
- moved R11 3.81 mm to (16.5, 16.5)
- moved R15 3.81 mm to (16.5, 26.7)
- moved R9 3.81 mm to (16.5, 29.2)
- moved C4 3.81 mm to (25.4, 8.89)
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Connections:
- net +5V: now also C11.1, C12.1, C13.1, C14.1, C15.1, C16.1, C17.1, U2.VBUS1
- net GND: now also C11.2, C12.2, C13.2, C14.2, C15.2, C16.2, C17.2, U2.GND1
Routing:
- net IRQ1: track 173.2 -> 123.7 mm, vias 2 -> 4
- net MEM_A16: track 104.2 -> 145.7 mm, vias 2 -> 1
- net +5V: track 261.2 -> 296.2 mm
- net MEM_A15: track 120.7 -> 150.9 mm, vias 3 -> 0
- net PAGE_FN1: track 106.1 -> 83.7 mm, vias 2 -> 1
- net A12: track 133.9 -> 112.9 mm, vias 0 -> 2
- net PAGE_FN3: track 89.8 -> 75.9 mm, vias 2 -> 1
- net PAGE_A17: track 82.0 -> 68.8 mm, vias 0 -> 1
- net PAGE_A15: track 108.1 -> 95.8 mm
- net RW: track 90.6 -> 78.3 mm, vias 2 -> 1
- net PAGE_A16: track 100.8 -> 88.6 mm
- net PAGE_A14: track 95.7 -> 84.0 mm, vias 1 -> 0
- net A9: track 79.1 -> 89.5 mm, vias 0 -> 1
- net E: track 88.4 -> 78.6 mm, vias 3 -> 1
- net A7: track 129.7 -> 138.5 mm
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Other:
- board text added: "POWER IN"

Commit message: updated
Parts:
- flipped R16 to the bottom, turned to 0 degrees
Routing:
- net MEM_A15: track 150.9 -> 111.1 mm, vias 0 -> 5
- net MEM_A16: track 145.7 -> 115.0 mm, vias 1 -> 3
- net PAGE_A15: track 95.8 -> 85.0 mm, vias 1 -> 3
- net RAMCS: track 63.8 -> 73.9 mm
- net PAGE_FN3: track 75.9 -> 85.7 mm, vias 1 -> 3
- net MEM_A14: track 80.8 -> 71.5 mm, vias 6 -> 7
- net RES: track 117.0 -> 125.8 mm
- net A6: track 135.6 -> 144.3 mm, vias 2 -> 0
- net A12: track 112.9 -> 121.7 mm, vias 2 -> 0
- net A13: track 86.5 -> 78.3 mm, vias 0 -> 1
- net IRQ2: track 127.1 -> 134.5 mm, vias 4 -> 2
- net IRQ1: track 123.7 -> 130.0 mm
- net RW: track 78.3 -> 83.4 mm, vias 1 -> 3
- net E: track 78.6 -> 83.0 mm, vias 1 -> 2
- net WR: track 154.7 -> 158.8 mm, vias 2 -> 1
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Other:
- board text added: "IN 5V"
- board text removed: "POWER IN"
